File: Sequencer/V02/Sequencer-V02-023.brd (EAGLE design)
At the start: 100 x 48 mm, 44 parts, among them IC2 LD117ADT50TR, IC6 LM1117MPX-ADJ, Q1 IRF530, X1 MARTIN8X2-1751303, X2 MARTIN3X2-1751303175L303-3, X3 MARTIN8X2-1751303, X4 1751264, X5 MARTIN3X2-1751303175L303-3

Commit message: V02 Final
Parts:
- removed JP1, JP3: JUMPER-SMT_2_NC_PASTE_NO-SILK, SparkFun-Jumpers:SMT-JUMPER_2_NC_PASTE_NO-SILK
- removed LED1, LED3, LED4, LED5, LED6: (no value), led:LED3MM
- added LED-BIAS, LED-LNA, LED-PA, LED-TRV, LED-TRX: (no value), led:LED3MM
- D3: device diode:D-2.5 -> diode:D-7.5
- R1, R3, R4, R5, R6, R7: device rcl:0204/5 -> rcl:0207/7
- moved Q1 91.1 mm to (13.9, 0.36), turned to 180 degrees
- moved R7 78.3 mm to (17.1, 11.4), turned to 270 degrees
- moved C11 10.0 mm to (12.7, 19.1), turned to 180 degrees
- moved RAW2 5.85 mm to (63.1, 22.2)
- moved C4 5.75 mm to (54.0, 10.8), flipped to the top
- moved IC2 5.75 mm to (13.0, 30.5)
- moved IC6 5.75 mm to (13.0, 30.5)
- moved C6 4.87 mm to (12.7, 22.2), flipped to the top, turned to 180 degrees
- moved D3 3.81 mm to (14.6, 11.4), turned to 270 degrees
- moved F2 3.18 mm to (10.2, 12.7), turned to 270 degrees
- moved JP2 3.18 mm to (10.2, 12.7), turned to 270 degrees
- moved STEPDWN 1.80 mm to (1.91, 27.7)
- moved C2 1.27 mm to (58.4, 36.2)
- moved C7 1.27 mm to (34.3, 36.2)
- moved C8 0.64 mm to (26.0, 36.2)
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Connections:
- net N$5 renamed R1COM
- net N$6 renamed R2NO
- net N$8 renamed R1NO
- net N$9 renamed R1NC
- removed net N$2: REL2.COM, X2.1
- removed net N$4: JP3.2, X4.2
- removed net N$7: REL2.NC, X2.3
- new net R2COM: REL2.COM, X2.3
- new net R2NC: REL2.NC, X2.1
- net BIAS-LED: now also LED-BIAS.K; no longer LED5.K
- net D8: no longer JP1.1
- net D9: no longer JP3.1
- net GND: now also LED-LNA.K; no longer LED1.K
- net LNA-LED: now also LED-LNA.A; no longer LED1.A
- net N$3: no longer JP1.2
- net PA-LED: now also LED-PA.K; no longer LED6.K
- net TRV-LED: now also LED-TRV.K; no longer LED4.K
- net TRX-LED: now also LED-TRX.K; no longer LED3.K
- net VCC: now also LED-BIAS.A, LED-PA.A, LED-TRV.A, LED-TRX.A; no longer LED3.A, LED4.A, LED5.A, LED6.A
Routing:
- net GND: track 0.00 -> 217.7 mm, vias 0 -> 43
- net VCC: track 0.00 -> 206.6 mm
- net UREG: track 0.00 -> 116.1 mm
- net 12V-LNA: track 0.00 -> 93.1 mm, vias 0 -> 1
- net BIASPA: track 0.00 -> 78.7 mm
- net D7: track 0.00 -> 74.2 mm
- net D6: track 0.00 -> 71.6 mm
- net D5: track 0.00 -> 69.8 mm
- net RELAIS-PA: track 0.00 -> 63.9 mm
- net D9: track 0.00 -> 57.4 mm
- net D8: track 0.00 -> 55.5 mm
- net LNA-LED: track 0.00 -> 51.4 mm
- net D4: track 0.00 -> 49.1 mm
- net D3: track 0.00 -> 48.6 mm
- net PA-LED: track 0.00 -> 43.1 mm
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Other:
- board text added: "COM"
- board text added: "NC"
- board text added: "NOpen"
- board text added: "Relais!"
- board text added: "Relais2"
- board text added: "TRV"
- board text removed: "VCC / VIN"
- board text removed: "VDD-Select"
