File: Sequencer/V02/Sequencer-V02-023.sch (EAGLE design)
At the start: 44 parts, among them IC2 LD117ADT50TR, IC6 LM1117MPX-ADJ, Q1 IRF530, X1 MARTIN8X2-1751303, X2 MARTIN3X2-1751303175L303-3, X3 MARTIN8X2-1751303, X4 1751264, X5 MARTIN3X2-1751303175L303-3

Commit message: V02 Final
Parts:
- removed JP1, JP3: JUMPER-SMT_2_NC_PASTE_NO-SILK, SparkFun-Jumpers:JUMPER-SMT_2_NC_PASTE_NO-SILK
- D3: device diode:DIODE-D-2.5 -> diode:DIODE-D-7.5
- R1, R3, R4, R5, R6, R7: device rcl:R-EU_0204/5 -> rcl:R-EU_0207/7
- renumbered LED1 to LED-LNA, LED3 to LED-TRX, LED4 to LED-TRV, LED5 to LED-BIAS, LED6 to LED-PA
Connections:
- net N$5 renamed R1COM
- net N$6 renamed R2NO
- net N$8 renamed R1NO
- net N$9 renamed R1NC
- removed net N$2: REL22.P, X2-1.K
- removed net N$4: JP3.2, X4-2.K
- removed net N$7: REL22.O, X2-3.K
- new net R2COM: REL22.P, X2-3.K
- new net R2NC: REL22.O, X2-1.K
- net D8: no longer JP1.1
- net D9: no longer JP3.1
- net N$3: no longer JP1.2
Other:
- moved on the sheet: C1, C2, X1-5, X1-7, X2-1, X2-3
