File: Sequencer/V02/Sequencer-V02-025.brd (EAGLE design)
At the start: 100 x 48 mm, 42 parts, among them IC2 LD117ADT50TR, IC6 LM1117MPX-ADJ, Q1 IRF530, X1 MARTIN8X2-1751303, X2 MARTIN3X2-1751303175L303-3, X3 MARTIN8X2-1751303, X4 1751264, X5 MARTIN3X2-1751303175L303-3

Commit message: v92
Connections:
- removed net N$3: X4.3
- net VIN: now also X4.3
Routing:
- net VIN: track 22.5 -> 23.9 mm
Other:
- board text added: "10K"
- board text added: "Fuse or Bridge"
- board text added: "MysX Connector"
- board text added: "NO"
- board text added: "Relais1"
- board text added: "Sequencer V0.2 (C) www.neuby.de"
- board text removed: "* = or Bridge"
- board text removed: "Fuse*"
- board text removed: "NOpen"
- board text removed: "Relais!"
Changed lines of the file:
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@@
 <grid distance="25" unitdist="mil" unit="mil" style="lines" multiple="1" display="yes" altdistance="0.1" altunitdist="mm" altunit="mm"/>
 <layers>
-<layer number="1" name="Top" color="4" fill="1" visible="no" active="yes"/>
+<layer number="1" name="Top" color="4" fill="1" visible="yes" active="yes"/>
 <layer number="2" name="Route2" color="1" fill="3" visible="no" active="no"/>
 <layer number="3" name="Route3" color="4" fill="3" visible="no" active="no"/>
@@
 <layer number="14" name="Route14" color="1" fill="6" visible="no" active="no"/>
 <layer number="15" name="Route15" color="4" fill="6" visible="no" active="no"/>
-<layer number="16" name="Bottom" color="1" fill="1" visible="yes" active="yes"/>
+<layer number="16" name="Bottom" color="1" fill="1" visible="no" active="yes"/>
 <layer number="17" name="Pads" color="2" fill="1" visible="yes" active="yes"/>
 <layer number="18" name="Vias" color="2" fill="1" visible="yes" active="yes"/>
 <layer number="19" name="Unrouted" color="6" fill="1" visible="yes" active="yes"/>
 <layer number="20" name="Dimension" color="15" fill="1" visible="yes" active="yes"/>
-<layer number="21" name="tPlace" color="7" fill="1" visible="no" active="yes"/>
-<layer number="22" name="bPlace" color="7" fill="1" visible="yes" active="yes"/>
-<layer number="23" name="tOrigins" color="15" fill="1" visible="no" active="yes"/>
-<layer number="24" name="bOrigins" color="15" fill="1" visible="yes" active="yes"/>
-<layer number="25" name="tNames" color="7" fill="1" visible="no" active="yes"/>
-<layer number="26" name="bNames" color="7" fill="1" visible="yes" active="yes"/>
+<layer number="21" name="tPlace" color="7" fill="1" visible="yes" active="yes"/>
+<layer number="22" name="bPlace" color="7" fill="1" visible="no" active="yes"/>
+<layer number="23" name="tOrigins" color="15" fill="1" visible="yes" active="yes"/>
+<layer number="24" name="bOrigins" color="15" fill="1" visible="no" active="yes"/>
+<layer number="25" name="tNames" color="7" fill="1" visible="yes" active="yes"/>
+<layer number="26" name="bNames" color="7" fill="1" visible="no" active="yes"/>
 <layer number="27" name="tValues" color="7" fill="1" visible="no" active="yes"/>
 <layer number="28" name="bValues" color="7" fill="1" visible="no" active="yes"/>
@@
 <layer number="37" name="tTest" color="7" fill="1" visible="no" active="yes"/>
 <layer number="38" name="bTest" color="7" fill="1" visible="no" active="yes"/>
-<layer number="39" name="tKeepout" color="4" fill="11" visible="no" active="yes"/>
-<layer number="40" name="bKeepout" color="1" fill="11" visible="yes" active="yes"/>
-<layer number="41" name="tRestrict" color="4" fill="10" visible="no" active="yes"/>
-<layer number="42" name="bRestrict" color="1" fill="10" visible="yes" active="yes"/>
+<layer number="39" name="tKeepout" color="4" fill="11" visible="yes" active="yes"/>
+<layer number="40" name="bKeepout" color="1" fill="11" visible="no" active="yes"/>
+<layer number="41" name="tRestrict" color="4" fill="10" visible="yes" active="yes"/>
+<layer number="42" name="bRestrict" color="1" fill="10" visible="no" active="yes"/>
 <layer number="43" name="vRestrict" color="2" fill="10" visible="no" active="yes"/>
 <layer number="44" name="Drills" color="7" fill="1" visible="no" active="yes"/>
@@
 <layer number="49" name="Reference" color="7" fill="1" visible="no" active="yes"/>
 <layer number="50" name="dxf" color="7" fill="1" visible="no" active="no"/>
-<layer number="51" name="tDocu" color="7" fill="1" visible="no" active="yes"/>
-<layer number="52" name="bDocu" color="7" fill="1" visible="yes" active="yes"/>
+<layer number="51" name="tDocu" color="7" fill="1" visible="yes" active="yes"/>
+<layer number="52" name="bDocu" color="7" fill="1" visible="no" active="yes"/>
 <layer number="53" name="tGND_GNDA" color="7" fill="9" visible="no" active="no"/>
 <layer number="54" name="bGND_GNDA" color="1" fill="9" visible="no" active="no"/>
@@
 <text x="3.175" y="7.62" size="0.8128" layer="26" font="vector" rot="MR0">VIN</text>
 <text x="12.573" y="46.482" size="0.8128" layer="26" font="vector" rot="MR180">Spare</text>
-<text x="23.368" y="42.672" size="0.8128" layer="26" font="vector" rot="MR180">TRX</text>
-<text x="17.018" y="42.672" size="0.8128" layer="26" font="vector" rot="MR180">Trv</text>
+<text x="16.383" y="42.672" size="0.8128" layer="26" font="vector" rot="MR180">TRX</text>
+<text x="23.368" y="42.672" size="0.8128" layer="26" font="vector" rot="MR180">Trv</text>
 <text x="29.083" y="42.672" size="0.8128" layer="26" font="vector" rot="MR180">BIAS-PA</text>
 <text x="36.703" y="42.672" size="0.8128" layer="26" font="vector" rot="MR180">Ralais-PA</text>
@@
 <text x="82.55" y="31.115" size="0.8128" layer="25" font="vector">100p</text>
 <text x="13.97" y="20.955" size="0.8128" layer="25" font="vector" rot="R180">100p</text>
-<text x="8.89" y="8.89" size="0.8128" layer="25" font="vector">Fuse*</text>
-<text x="1.27" y="42.545" size="0.8128" layer="25" font="vector" rot="R270">* = or Bridge</text>
+<text x="8.89" y="6.35" size="0.8128" layer="25" font="vector">Fuse
+or
+Bridge</text>
 <text x="21.59" y="4.445" size="0.8128" layer="25" font="vector">VCC</text>
 <text x="24.13" y="4.445" size="0.8128" layer="25" font="vector">Spr</text>
@@
 <text x="42.545" y="1.27" size="2.032" layer="25" font="vector">LEDs</text>
 <text x="3.81" y="20.32" size="0.8128" layer="25" font="vector">GND</text>
-<text x="7.62" y="10.795" size="0.8128" layer="25" font="vector" rot="R90">D9</text>
-<text x="7.62" y="14.605" size="0.8128" layer="25" font="vector" rot="R90">D8</text>
 <text x="8.89" y="28.575" size="0.8128" layer="25" font="vector" rot="R90">Regulator</text>
 <text x="10.16" y="34.925" size="0.8128" layer="25" font="vector" rot="R90">+</text>
@@
 <text x="68.834" y="41.91" size="0.8128" layer="26" font="vector" rot="MR180">Relais2</text>
 <text x="73.914" y="46.355" size="0.8128" layer="26" font="vector" rot="MR180">COM</text>
-<text x="69.469" y="46.355" size="0.8128" layer="26" font="vector" rot="MR180">NOpen</text>
+<text x="70.104" y="46.355" size="0.8128" layer="26" font="vector" rot="MR180">NO</text>
 <text x="66.929" y="46.355" size="0.8128" layer="26" font="vector" rot="MR180">NC</text>
 <text x="77.089" y="46.355" size="0.8128" layer="26" font="vector" rot="MR180">COM</text>
-<text x="80.264" y="46.355" size="0.8128" layer="26" font="vector" rot="MR180">NOpen</text>
-<text x="84.709" y="46.355" size="0.8128" layer="26" font="vector" rot="MR180">COM</text>
+<text x="80.899" y="46.355" size="0.8128" layer="26" font="vector" rot="MR180">NO</text>
+<text x="84.709" y="46.355" size="0.8128" layer="26" font="vector" rot="MR180">NC</text>
 <wire x1="78.105" y1="42.545" x2="86.995" y2="42.545" width="0.254" layer="26"/>
-<text x="80.264" y="41.91" size="0.8128" layer="26" font="vector" rot="MR180">Relais!</text>
+<text x="80.264" y="41.91" size="0.8128" layer="26" font="vector" rot="MR180">Relais1</text>
 <text x="23.495" y="31.115" size="0.8128" layer="25" font="vector" rot="R90">TRX</text>
 <text x="30.48" y="31.115" size="0.8128" layer="25" font="vector" rot="R90">TRV</text>
@@
 <text x="45.085" y="31.115" size="0.8128" layer="25" font="vector" rot="R90">PA</text>
 <text x="51.435" y="30.48" size="0.8128" layer="25" font="vector" rot="R90">LNA</text>
+<text x="6.915" y="16.335" size="1.016" layer="25" rot="R270">VIn</text>
+<text x="6.915" y="9.35" size="1.016" layer="25" rot="R270">VIn</text>
+<text x="3.175" y="14.605" size="0.8128" layer="26" font="vector" rot="MR0">VIN</text>
+<text x="19.05" y="8.89" size="0.8128" layer="25" font="vector" rot="R90">10K</text>
+<text x="66.04" y="6.985" size="0.8128" layer="25" font="vector">MysX Connector</text>
+<text x="43.18" y="20.32" size="0.8128" layer="25" font="vector">Sequencer V0.2
+(C) www.neuby.de</text>
 </plain>
 <attributes>
@@
 </element>
 <element name="R7" library="rcl" library_urn="urn:adsk.eagle:library:334" package="0207/7" package3d_urn="urn:adsk.eagle:package:23493/2" value="10K" x="17.145" y="11.43" smashed="yes" rot="R270">
-<attribute name="NAME" x="18.313396875" y="13.4366" size="0.9906" layer="25" ratio="10" rot="R270"/>
+<attribute name="NAME" x="18.415" y="13.335" size="0.9906" layer="25" ratio="10" rot="R270"/>
 <attribute name="POPULARITY" value="46" x="17.145" y="11.43" size="1.778" layer="27" rot="R270" display="off"/>
 <attribute name="SPICEPREFIX" value="R" x="17.145" y="11.43" size="1.778" layer="27" rot="R270" display="off"/>
@@
 <wire x1="10.16" y1="11.3" x2="10.16" y2="12.1694" width="0.6348" layer="1"/>
 <wire x1="13.97" y1="19.05" x2="12.8015" y2="19.05" width="0.762" layer="1"/>
+<contactref element="X4" pad="3"/>
+<wire x1="4.77" y1="15.335" x2="4.77" y2="14.1364" width="0.762" layer="1"/>
+<wire x1="4.77" y1="14.1364" x2="4.9575" y2="13.9489" width="0.762" layer="1"/>
 </signal>
 <signal name="RX0" class="2">
@@
 <wire x1="20.5996" y1="17.2975" x2="21.59" y2="17.2975" width="1.2192" layer="1"/>
 </signal>
-<signal name="N$3">
-<contactref element="X4" pad="3"/>
-</signal>
 <signal name="R2COM">
