File: Sequencer/V02/Sequencer-V02-023e.brd (EAGLE design)
At the start: 100 x 48 mm, 42 parts, among them IC2 LD117ADT50TR, IC6 LM1117MPX-ADJ, Q1 IRF530, X1 MARTIN8X2-1751303, X2 MARTIN3X2-1751303175L303-3, X3 MARTIN8X2-1751303, X4 1751264, X5 MARTIN3X2-1751303175L303-3

Commit message: Sequencer V1.0
Routing:
- net VCC: track 206.6 -> 184.7 mm
- net 12V-LNA: track 93.1 -> 106.6 mm, vias 1 -> 0
- net GND: track 217.7 -> 209.6 mm, vias 43 -> 42
- net D7: track 74.2 -> 67.9 mm
- net D8: track 55.5 -> 60.3 mm
- net D5: track 69.8 -> 65.2 mm
- net VIN: track 23.9 -> 27.2 mm
- net D6: track 71.6 -> 68.6 mm
- net MOSFET: track 22.1 -> 20.1 mm
- net D9: track 57.4 -> 55.4 mm
- net D4: track 49.1 -> 51.0 mm
- net R1NC: track 14.5 -> 15.7 mm, vias 0 -> 1
- net A7: track 20.9 -> 21.6 mm
- net RELAIS-PA: track 63.9 -> 63.2 mm
- net UREG: track 116.1 -> 115.4 mm
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Other:
- board text added: "Relais-PA"
- board text added: "ULN"
- board text removed: "10K"
- board text removed: "MysX Connector"
- board text removed: "Ralais-PA"
- board text removed: "Sequencer V0.2 (C) www.neuby.de"
