File: Sequencer/V02/Sequencer-V02-023e.sch (EAGLE design)
At the start: 42 parts, among them IC2 LD117ADT50TR, IC6 LM1117MPX-ADJ, Q1 IRF530, X1 MARTIN8X2-1751303, X2 MARTIN3X2-1751303175L303-3, X3 MARTIN8X2-1751303, X4 1751264, X5 MARTIN3X2-1751303175L303-3

Commit message: Sequencer V1.0
Changed lines of the file:
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@@
 <pinref part="X1" gate="-5" pin="K"/>
+</segment>
+<segment>
+<wire x1="-58.42" y1="21.59" x2="-52.07" y2="21.59" width="0.1524" layer="91"/>
+<label x="-52.07" y="21.59" size="1.778" layer="95" xref="yes"/>
 </segment>
 </net>
@@
 <junction x="134.62" y="129.54"/>
 <pinref part="X1" gate="-7" pin="K"/>
+</segment>
+<segment>
+<wire x1="-68.58" y1="19.05" x2="-52.07" y2="19.05" width="0.1524" layer="91"/>
+<label x="-52.07" y="19.05" size="1.778" layer="95" xref="yes"/>
 </segment>
 </net>
@@
 <net name="VIN" class="1">
 <segment>
-<wire x1="-78.74" y1="16.51" x2="-72.39" y2="16.51" width="0.1524" layer="91"/>
+<wire x1="-78.74" y1="16.51" x2="-68.58" y2="16.51" width="0.1524" layer="91"/>
 <label x="-78.74" y="16.51" size="1.778" layer="95"/>
 <pinref part="X4" gate="-1" pin="K"/>
-<pinref part="X4" gate="-3" pin="K"/>
-<wire x1="-72.39" y1="16.51" x2="-68.58" y2="16.51" width="0.1524" layer="91"/>
-<wire x1="-68.58" y1="21.59" x2="-72.39" y2="21.59" width="0.1524" layer="91"/>
-<wire x1="-72.39" y1="21.59" x2="-78.74" y2="21.59" width="0.1524" layer="91"/>
-<wire x1="-72.39" y1="21.59" x2="-72.39" y2="16.51" width="0.1524" layer="91"/>
-<junction x="-72.39" y="21.59"/>
 </segment>
 <segment>
@@
 <label x="-86.36" y="58.42" size="1.778" layer="95" rot="R180" xref="yes"/>
 </segment>
+<segment>
+<pinref part="X4" gate="-3" pin="K"/>
+<wire x1="-68.58" y1="21.59" x2="-78.74" y2="21.59" width="0.1524" layer="91"/>
+<label x="-78.74" y="21.59" size="1.778" layer="95"/>
+</segment>
 </net>
